File: circuit/bedheater.kicad_pcb (KiCad board)
At the start: 2 copper layers, 20 parts, among them CON1 AVR-ISP-6, CON2 BARREL_JACK, IC1 ATMEGA328-P, P1 Heater+, P2 CONN_01X02, P3 Heater-, Q1 TIP142, U1 OKI-78SR-3.3, U2 UB232R, Y1 20 MHz

Commit message: Update PID params. Fix schematic/pcb issue where the TIP142 was connected as though it were PNP (it is an NPN BJT). Correct some connectivity issues in the app
Parts:
- added R5: 10K, Resistors_ThroughHole:Resistor_Horizontal_RM10mm, F.Cu at (153.2, 82.3)
- moved P3 17.1 mm to (207.3, 81.5)
- moved P1 13.2 mm to (194.3, 81.5)
Connections:
- IC1 pad 4: /heater -> (no net)
- IC1 pad 5: (no net) -> /heater
- P1 pad 1: Net-(P1-Pad1) -> +12V
- P3 pad 1: GND -> Net-(P3-Pad1)
- Q1 pad 2: +12V -> Net-(P3-Pad1)
- Q1 pad 3: Net-(P1-Pad1) -> GND
Routing:
- net +3V3: track 79.1 -> 84.9 mm
- net /RST: track 41.4 -> 46.0 mm
- net /heater: track 56.7 -> 59.4 mm
- added copper zone on B.Cu, net Net-(P3-Pad1)
- removed copper zone on B.Cu, net Net-(P1-Pad1)
